Commit message: ficheros de simulacion

File: Humanoide/codigo/humanoide.urdf (robot description, URDF)
Before this commit: robot humanoide, 17 links, 16 joints
Links:
- removed link bod
- removed link brazo.der
- removed link brazo.izq
- removed link hombro.der
- removed link hombro.izq
- removed link mano.der
- removed link mano.izq
- removed link pie.der
- removed link pie.izq
- removed link pierna.d1
- removed link pierna.d2
- removed link pierna.d3
- removed link pierna.d4
- removed link pierna.i1
- removed link pierna.i2
- removed link pierna.i3
- removed link pierna.i4
- added link base, mass 0.0001
- added link chest, mass 14.000000; collision sphere radius=0.440000
- added link left_ankle, mass 1.000000; collision box size=0.708000 0.220000 0.360000
- added link left_elbow, mass 1.000000; collision capsule length=0.540000 radius=0.160000
- added link left_hip, mass 4.500000; collision capsule length=1.200000 radius=0.220000
- added link left_knee, mass 3.000000; collision capsule length=1.240000 radius=0.200000
- added link left_shoulder, mass 1.500000; collision capsule length=0.720000 radius=0.180000
- added link left_wrist, mass 0.500000; collision sphere radius=0.160000
- added link neck, mass 2.000000; collision sphere radius=0.410000
- added link right_ankle, mass 1.000000; collision box size=0.708000 0.220000 0.360000
- added link right_elbow, mass 1.000000; collision capsule length=0.540000 radius=0.160000
- added link right_hip, mass 4.500000; collision capsule length=1.200000 radius=0.220000
- added link right_knee, mass 3.000000; collision capsule length=1.240000 radius=0.200000
- added link right_shoulder, mass 1.500000; collision capsule length=0.720000 radius=0.180000
- added link right_wrist, mass 0.500000; collision sphere radius=0.160000
- added link root, mass 6.000000; collision sphere radius=0.360000
Joints:
- removed joint ankle_forwards.d
- removed joint ankle_forwards.i
- removed joint ankle_side.d
- removed joint ankle_side.i
- removed joint arm_pitch.d
- removed joint arm_pitch.i
- removed joint arm_roll.d
- removed joint arm_roll.i
- removed joint hip_roll.d
- removed joint hip_roll.i
- removed joint leg_forwards.d
- removed joint leg_forwards.i
- removed joint leg_side.d
- removed joint leg_side.i
- removed joint wrist.d
- removed joint wrist.i
- added joint chest: type spherical, parent root, child chest, origin xyz=0.000000 0.944604 0.000000 rpy=0 0 0
- added joint left_ankle: type spherical, parent left_knee, child left_ankle, origin xyz=0.000000 -1.639480 0.000000 rpy=0 0 0
- added joint left_elbow: type revolute, parent left_shoulder, child left_elbow, origin xyz=0.000000 -1.099152 0.000000 rpy=0 0 0, axis 0.000000 0.000000 1.000000, limit lower=0 upper=3.14 effort=1000.0 velocity=0.5
- added joint left_hip: type spherical, parent root, child left_hip, origin xyz=0.000000 0.000000 -0.339548 rpy=0 0 0
- added joint left_knee: type revolute, parent left_hip, child left_knee, origin xyz=0.000000 -1.686184 0.000000 rpy=0 0 0, axis 0.000000 0.000000 1.000000, limit lower=-3.14 upper=0. effort=1000.0 velocity=0.5
- added joint left_shoulder: type spherical, parent chest, child left_shoulder, origin xyz=-0.096200 0.974000 -0.732440 rpy=0 0 0
- added joint left_wrist: type fixed, parent left_elbow, child left_wrist, origin xyz=0.000000 -1.035788 0.000000 rpy=0 0 0
- added joint neck: type spherical, parent chest, child neck, origin xyz=0.000000 0.895576 0.000000 rpy=0 0 0
- added joint right_ankle: type spherical, parent right_knee, child right_ankle, origin xyz=0.000000 -1.639480 0.000000 rpy=0 0 0
- added joint right_elbow: type revolute, parent right_shoulder, child right_elbow, origin xyz=0.000000 -1.099152 0.000000 rpy=0 0 0, axis 0.000000 0.000000 1.000000, limit lower=0 upper=3.14 effort=1000.0 velocity=0.5
- added joint right_hip: type spherical, parent root, child right_hip, origin xyz=0.000000 0.000000 0.339548 rpy=0 0 0
- added joint right_knee: type revolute, parent right_hip, child right_knee, origin xyz=0.000000 -1.686184 0.000000 rpy=0 0 0, axis 0.000000 0.000000 1.000000, limit lower=-3.14 upper=0. effort=1000.0 velocity=0.5
- added joint right_shoulder: type spherical, parent chest, child right_shoulder, origin xyz=-0.096200 0.974000 0.732440 rpy=0 0 0
- added joint right_wrist: type fixed, parent right_elbow, child right_wrist, origin xyz=0.000000 -1.035788 0.000000 rpy=0 0 0
- added joint root: type fixed, parent base, child root, origin xyz=0.000000 0.000000 0.000000 rpy=0 0 0
