File: Torreta/pcb/AmplificadorV1/AmplificadorV1.kicad_pcb (KiCad board)
At the start: 2 copper layers, 4 parts, among them J1 Conn_Coaxial, J2 Conn_01x02_Female, J3 Conn_Coaxial, U1 Amplificador_2_4Ghz

Commit message: nueva placa
Parts:
- added  : MountingHole_3.2mm_M3, MountingHole:MountingHole_3.2mm_M3, F.Cu at (160.0, 109.2)
- added  : MountingHole_3.2mm_M3, MountingHole:MountingHole_3.2mm_M3, F.Cu at (144.5, 85.6)
- added  : MountingHole_3.2mm_M3, MountingHole:MountingHole_3.2mm_M3, F.Cu at (175.3, 85.9)
- added 0.1uF1: C, Capacitor_SMD:C_0402_1005Metric, F.Cu at (164.2, 93.6)
- added 1.8pF1: C, Capacitor_SMD:C_0603_1608Metric, F.Cu at (154.3, 102.4)
- added 100pF1: C, Capacitor_SMD:C_0805_2012Metric, F.Cu at (164.7, 96.0)
- added 15nH1: INDUCTOR, Inductor_SMD:L_0402_1005Metric, F.Cu at (164.0, 101.1)
- added 18pF1: C, Capacitor_SMD:C_1206_3216Metric, F.Cu at (167.7, 101.6)
- added 2.0pF1: C, Capacitor_SMD:C_0805_2012Metric, F.Cu at (151.6, 101.6)
- added 33nH1: INDUCTOR, Inductor_SMD:L_0402_1005Metric, F.Cu at (148.8, 102.1)
- added R1: 7.5K, Resistor_SMD:R_0603_1608Metric, F.Cu at (155.7, 96.8)
- J1, J3: footprint Connector_Coaxial:SMA_Amphenol_132289_EdgeMount -> Connector_Coaxial:SMA_Samtec_SMA-J-P-X-ST-EM1_EdgeMount
- U1: footprint FootprintAmpli:QFN50P350X350X100-17N -> Package_DFN_QFN:QFN-16-1EP_3x3mm_P0.5mm_EP1.75x1.75mm
- moved J1 271.6 mm to (144.8, 101.6), turned to 270 degrees
- moved J2 242.2 mm to (159.5, 87.9)
- moved U1 242.1 mm to (159.7, 101.0)
- moved J3 208.4 mm to (174.8, 101.6), turned to 90 degrees
Connections:
- J1 pad 1: Net-(J1-Pad1) -> señal
- J1 pad 2: Net-(J1-Pad2) -> GND
- J2 pad 1: Net-(J2-Pad1) -> VDD
- J2 pad 2: Net-(J2-Pad2) -> GND
- J3 pad 1: Net-(J3-Pad1) -> Net-(18pF1-Pad1)
- J3 pad 2: Net-(J3-Pad2) -> GND
- U1 pad 10: Net-(J3-Pad1) -> señal
- U1 pad 3: Net-(J1-Pad1) -> Net-(1.8pF1-Pad1)
- U1 pad 4: Net-(J1-Pad1) -> Net-(1.8pF1-Pad1)
- U1 pad 9: Net-(J3-Pad1) -> señal
Routing:
- net Net-(J3-Pad1): track 57.3 -> 0.00 mm
- net GND: track 0.00 -> 43.8 mm, vias 0 -> 19
- net VDD: track 0.00 -> 24.3 mm
- net señal: track 0.00 -> 11.7 mm
- net Net-(1.8pF1-Pad1): track 0.00 -> 6.21 mm
- net Net-(18pF1-Pad1): track 0.00 -> 5.81 mm
- net Net-(R1-Pad1): track 0.00 -> 3.66 mm
- net Net-(U1-Pad5): track 0.00 -> 1.72 mm, vias 0 -> 1
- net Net-(U1-Pad16): track 0.00 -> 1.41 mm, vias 0 -> 1
- net Net-(U1-Pad8): track 0.00 -> 1.39 mm, vias 0 -> 1
- net Net-(U1-Pad13): track 0.00 -> 1.37 mm, vias 0 -> 1
- net Net-(U1-Pad12): track 0.00 -> 1.34 mm, vias 0 -> 1
- net Net-(U1-Pad6): track 0.00 -> 1.32 mm, vias 0 -> 1
- net Net-(U1-Pad15): track 0.00 -> 1.20 mm, vias 0 -> 1
- net Net-(U1-Pad11): track 0.00 -> 1.18 mm, vias 0 -> 1
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- added copper zone on In1.Cu, net GND
- added copper zone on In2.Cu, net GND
Other:
- board outline added: 35.3 x 34.3 mm
- copper layers 2 -> 4
- net class señal added: clearance 0.2, trace_width 0.29337, via_dia 0.8, via_drill 0.4
- board text added: "10V"
- board text added: "GND"
- board text added: "RFin"
- board text added: "RFout"
- board text added: "Raúl González"
- board text added: "V1.0"
