File: Torreta/pcb/AmplificadorV1/AmplificadorV1.kicad_pcb (KiCad board)
At the start: 4 copper layers, 35.3 x 34.3 mm, 15 parts, among them J1 Conn_Coaxial, J2 Conn_01x02_Female, J3 Conn_Coaxial, U1 Amplificador_2_4Ghz

Commit message: Revisión placa y atenuadores
Parts:
- removed the   at (160.0, 109.2)
- removed the   at (175.3, 85.9)
- moved 33nH1 3.20 mm to (152.0, 102.1)
- moved 2.0pF1 2.82 mm to (154.4, 101.7)
- moved 1.8pF1 2.62 mm to (156.9, 102.4)
- moved 18pF1 2.46 mm to (165.3, 101.7)
- moved 15nH1 1.60 mm to (162.4, 101.2)
Routing:
- net GND: track 43.8 -> 19.5 mm, vias 19 -> 5
- net señal: track 11.7 -> 1.46 mm
- net Net-(1.8pF1-Pad1): track 6.21 -> 0.00 mm
- net VDD: track 24.3 -> 20.0 mm
- net Net-(18pF1-Pad1): track 5.81 -> 8.30 mm
- net Net-(U1-Pad12): track 1.34 -> 0.00 mm, vias 1 -> 0
- net Net-(U1-Pad11): track 1.18 -> 0.00 mm, vias 1 -> 0
- net Net-(U1-Pad2): track 1.03 -> 0.00 mm, vias 1 -> 0
Other:
- outline, holes or cut-outs redrawn
