File: Torreta/pcb/AmplificadorV1/AmplificadorV2.kicad_pcb (KiCad board)
At the start: 4 copper layers, 35.3 x 34.3 mm, 15 parts, among them J1 Conn_Coaxial, J2 Conn_01x02_Female, J3 Conn_Coaxial, U1 Amplificador_2_4Ghz

Commit message: Revisión placa y atenuadores
Parts:
- removed the   at (160.0, 109.2)
- removed the   at (175.3, 85.9)
- removed 33nH1: INDUCTOR, Inductor_SMD:L_0402_1005Metric
- added  : MountingHole_3.2mm_M3, MountingHole:MountingHole_3.2mm_M3, F.Cu at (172.1, 109.2)
- added  : MountingHole_3.2mm_M3, MountingHole:MountingHole_3.2mm_M3, F.Cu at (146.6, 109.2)
- added  : MountingHole_3.2mm_M3, MountingHole:MountingHole_3.2mm_M3, F.Cu at (172.1, 85.5)
- moved 2.0pF1 3.13 mm to (154.7, 101.6)
- moved 1.8pF1 2.62 mm to (156.9, 102.3)
- moved   2.08 mm to (146.6, 85.5)
Routing:
- net GND: track 43.8 -> 18.7 mm, vias 19 -> 5
- net señal: track 11.7 -> 0.03 mm
- net Net-(1.8pF1-Pad1): track 6.21 -> 0.00 mm
- net Net-(18pF1-Pad1): track 5.81 -> 0.00 mm
- net Net-(U1-Pad2): track 1.03 -> 0.00 mm, vias 1 -> 0
Other:
- board size 35.3 x 34.3 mm -> 35.4 x 34.3 mm
